File: qspi-pmod.kicad_pcb (KiCad board)
At the start: 2 copper layers, 22.7 x 20 mm, 10 parts, among them J1 PMOD, U1 W25Q128JVS, U2 878-APS6404L-3SQR-SN, U3 878-APS6404L-3SQR-SN

Commit message: Finish routing
Parts:
- moved C6 7.65 mm to (160.3, 92.2), turned to 180 degrees
- moved C4 7.36 mm to (153.9, 92.2), turned to 180 degrees
- moved C5 7.27 mm to (160.3, 91.1), turned to 180 degrees
- moved C3 6.65 mm to (153.9, 91.1), turned to 180 degrees
- moved U2 2.94 mm to (152.5, 86.8), turned to -90 degrees
- moved U3 2.91 mm to (158.8, 86.8), turned to -90 degrees
- moved C2 2.12 mm to (161.0, 77.5)
- moved C1 2.08 mm to (159.9, 77.5)
- moved U1 0.80 mm to (154.5, 78.9)
- moved J1 0.24 mm to (147.0, 78.4)
Routing:
- net PMOD6: track 0.00 -> 52.3 mm
- net PMOD2: track 0.00 -> 36.9 mm, vias 0 -> 2
- net PMOD5: track 0.00 -> 28.7 mm, vias 0 -> 3
- net PMOD4: track 0.00 -> 26.6 mm
- net PMOD3: track 0.00 -> 23.9 mm, vias 0 -> 3
- net PMOD8: track 0.00 -> 18.8 mm, vias 0 -> 1
- net +3.3V: track 0.00 -> 12.5 mm
- net PMOD7: track 0.00 -> 12.2 mm, vias 0 -> 1
- net GND: track 0.00 -> 10.8 mm, vias 0 -> 6
- net PMOD1: track 0.00 -> 4.48 mm
- added copper zone on F.Cu, net +3.3V

Commit message: Fixup
Changed lines of the file:
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@@
     (property "ki_keywords" "PSRAM memory SPI")
     (attr smd)
-    (fp_text reference "U2" (at 2.9 3.395 90) (layer "F.SilkS")
+    (fp_text reference "U2" (at 4.6 1.895 90) (layer "F.SilkS")
         (effects (font (size 0.8 0.8) (thickness 0.1)))
     )
@@
     (property "ki_keywords" "connector")
     (attr through_hole)
-    (fp_text reference "J1" (at -5.655 -2.27) (layer "F.SilkS")
+    (fp_text reference "J1" (at -5.3 -2.27) (layer "F.SilkS")
         (effects (font (size 1 1) (thickness 0.15)))
     )
@@
     (property "ki_keywords" "PSRAM memory SPI")
     (attr smd)
-    (fp_text reference "U3" (at 2.9 -3.3 90) (layer "F.SilkS")
+    (fp_text reference "U3" (at 4.6 2 90) (layer "F.SilkS")
         (effects (font (size 0.8 0.8) (thickness 0.1)))
     )
@@
   (gr_line (start 162.7 93.7) (end 162.7 75.7)
     (stroke (width 0.1) (type default)) (layer "Edge.Cuts"))
-  (gr_text "${TITLE} ${REVISION}" (at 140.4 94.1) (layer "F.SilkS")
+  (gr_text "${TITLE} ${REVISION}" (at 140.8 93.9) (layer "F.SilkS")
     (effects (font (size 0.8 0.8) (thickness 0.15)) (justify left bottom))
   )
@@
   (segment (start 154.312201 80.4) (end 151.887701 82.8245) (width 0.25) (layer "B.Cu") (net 7))
   (segment (start 154.312201 80.4) (end 155.763201 80.4) (width 0.25) (layer "B.Cu") (net 7))
+  (segment (start 144.5 75.5) (end 153.7 75.5) (width 0.25) (layer "F.Cu") (net 8))
   (segment (start 142.9 79.38) (end 142.9 77.1) (width 0.25) (layer "F.Cu") (net 8))
   (segment (start 150.1 90.7) (end 152.754999 90.7) (width 0.25) (layer "F.Cu") (net 8))
@@
   (segment (start 143.973299 89.925) (end 149.325 89.925) (width 0.25) (layer "F.Cu") (net 8))
   (segment (start 149.325 89.925) (end 150.1 90.7) (width 0.25) (layer "F.Cu") (net 8))
+  (segment (start 153.7 75.5) (end 156.465 78.265) (width 0.25) (layer "F.Cu") (net 8))
   (segment (start 156.970908 88) (end 157.54 88.569092) (width 0.25) (layer "F.Cu") (net 8))
   (segment (start 157.775 90.575) (end 159.025 90.575) (width 0.25) (layer "F.Cu") (net 8))
   (segment (start 143.285 89.236701) (end 143.973299 89.925) (width 0.25) (layer "F.Cu") (net 8))
-  (segment (start 153.6 75.4) (end 156.465 78.265) (width 0.25) (layer "F.Cu") (net 8))
-  (segment (start 142.9 77.1) (end 144.6 75.4) (width 0.25) (layer "F.Cu") (net 8))
   (segment (start 153.13 90.324999) (end 153.13 89.425) (width 0.25) (layer "F.Cu") (net 8))
   (segment (start 144.46 80.94) (end 143.285 82.115) (width 0.25) (layer "F.Cu") (net 8))
-  (segment (start 144.6 75.4) (end 153.6 75.4) (width 0.25) (layer "F.Cu") (net 8))
-  (segment (start 144.46 80.94) (end 142.9 79.38) (width 0.25) (layer "F.Cu") (net 8))
   (segment (start 152.754999 90.7) (end 153.13 90.324999) (width 0.25) (layer "F.Cu") (net 8))
-  (segment (start 156.465 78.265) (end 158.1 78.265) (width 0.25) (layer "F.Cu") (net 8))
   (segment (start 153.13 89.425) (end 153.13 88.600001) (width 0.25) (layer "F.Cu") (net 8))
+  (segment (start 142.9 77.1) (end 144.5 75.5) (width 0.25) (layer "F.Cu") (net 8))
   (segment (start 153.1 89.395) (end 153.13 89.425) (width 0.25) (layer "F.Cu") (net 8))
   (segment (start 153.730001 88) (end 156.970908 88) (width 0.25) (layer "F.Cu") (net 8))
+  (segment (start 144.46 80.94) (end 142.9 79.38) (width 0.25) (layer "F.Cu") (net 8))
+  (segment (start 156.465 78.265) (end 158.1 78.265) (width 0.25) (layer "F.Cu") (net 8))
   (segment (start 159.435 90.165) (end 159.435 89.425) (width 0.25) (layer "F.Cu") (net 8))
   (segment (start 153.13 88.600001) (end 153.730001 88) (width 0.25) (layer "F.Cu") (net 8))
